Commit message: Multi-robot test

File: beacon_gazebo_plugin/urdf/autonet_v1.xacro (robot description, xacro)
@@ -129,4 +129,13 @@
     <preserveFixedJoint>true</preserveFixedJoint>
   </gazebo>
+  <joint name="beacon_joint" type="fixed">
+    <axis xyz="0 1 0" />
+    <origin xyz="0 0 0.1" rpy="0 0 0"/>
+    <parent link="base_link"/>
+    <child link="beacon_link"/>
+  </joint>
+  <gazebo reference='beacon_joint'>
+    <preserveFixedJoint>true</preserveFixedJoint>
+  </gazebo>
 <!--  &lt;!&ndash; Camera &ndash;&gt;-->
   <link name="front_bumper_link">
@@ -173,4 +182,25 @@
   </link>
   <link name="receiver_link">
+    <pose>0 0 0 0 0 0</pose>
+    <collision>
+      <origin xyz="0 0 0" rpy="0 0 0"/>
+      <geometry>
+        <box size="0.02 0.02 0.04"/>
+      </geometry>
+    </collision>
+    <visual>
+      <origin xyz="0 0 0" rpy="0 0 0"/>
+      <geometry>
+        <box size="0.02 0.02 0.04"/>
+      </geometry>
+      <!--      <material name="green"/>-->
+    </visual>
+    <inertial>
+      <mass value="1e-5" />
+      <origin xyz="0 0 0" rpy="0 0 0"/>
+      <inertia ixx="1e-6" ixy="0" ixz="0" iyy="1e-6" iyz="0" izz="1e-6" />
+    </inertial>
+  </link>
+  <link name="beacon_link">
     <pose>0 0 0 0 0 0</pose>
     <collision>

File: beacon_gazebo_plugin/urdf/autonet_v1_gazebo.xacro (robot description, xacro)
@@ -14,5 +14,8 @@
   </gazebo>
   <gazebo reference="receiver_link">
-    <material>Gazebo/Blue</material>
+    <material>Gazebo/Orange</material>
+  </gazebo>
+  <gazebo reference="beacon_link">
+    <material>Gazebo/Purple</material>
   </gazebo>
   <gazebo>

Commit message: Contact sensor experiments

File: beacon_gazebo_plugin/urdf/autonet_v1.xacro (robot description, xacro)
@@ -15,4 +15,5 @@
     <!-- body -->
     <collision name="collision_chassis">
+      <origin rpy="0 0 0" xyz="-0.1 0 0"/>
       <geometry>
         <box size="0.295 0.295 0.05"/>

File: beacon_gazebo_plugin/urdf/autonet_v1_gazebo.xacro (robot description, xacro)
@@ -54,4 +54,22 @@
 <!--      <geom>front_bumper_geom</geom>-->
 <!--    </plugin>-->
+    <sensor name="contact_sensor" type="contact">
+      <contact>
+        <collision>front_bumper_col</collision>
+        <topic>/front_bumper</topic>
+      </contact>
+      <self_collide>true</self_collide>
+      <always_on>true</always_on>
+      <update_rate>1000.0</update_rate>
+      <selfCollide>true</selfCollide>
+      <alwaysOn>true</alwaysOn>
+      <updateRate>1000.0</updateRate>
+<!--      <plugin name="gazebo_ros_bumper_controller" filename="libgazebo_ros_bumper.so">-->
+<!--        <bumperTopicName>front_bumper</bumperTopicName>-->
+<!--        <frameName>world</frameName>-->
+<!--        <alwaysOn>true</alwaysOn>-->
+<!--        <updateRate>1000.0</updateRate>-->
+<!--      </plugin>-->
+    </sensor>
 <!--    <sensor:contact name="contact_sensor">-->
 <!--      <geom>front_bumper_link</geom>-->
