Commit message: -_-

File: beacon_gazebo_plugin/urdf/autonet_v1/autonet_v1.xacro (robot description, xacro)
@@ -100,16 +100,16 @@
    -->
   <xacro:link_wheel name="link_right_wheel" />
-  <xacro:joint_wheel name="joint_right_wheel" child="link_right_wheel" origin_xyz="0 0.16 -0.012" />
+  <xacro:joint_wheel name="joint_right_wheel" child="link_right_wheel" origin_xyz="0 0.16 -0.012" parent="base_link" />
   <xacro:link_wheel name="link_left_wheel" />
-  <xacro:joint_wheel name="joint_left_wheel" child="link_left_wheel" origin_xyz="0 -0.16 -0.012" />
+  <xacro:joint_wheel name="joint_left_wheel" child="link_left_wheel" origin_xyz="0 -0.16 -0.012" parent="base_link" />
   <joint name="front_bumper_joint" type="fixed">
     <axis xyz="0 1 0" />
     <origin xyz="0.08 0 0" rpy="0 0 0"/>
     <parent link="base_link"/>
-    <child link="front_bumper_link"/>
-  </joint>
-  <gazebo reference='front_bumper_joint'>
-    <preserveFixedJoint>true</preserveFixedJoint>
-  </gazebo>
+    <child link="link_front_bumper"/>
+  </joint>
+<!--  <gazebo reference='front_bumper_joint'>-->
+<!--    <preserveFixedJoint>true</preserveFixedJoint>-->
+<!--  </gazebo>-->
   <joint name="imu_joint" type="fixed">
     <axis xyz="0 1 0" />
@@ -140,7 +140,7 @@
   </gazebo>
 <!--  &lt;!&ndash; Camera &ndash;&gt;-->
-  <link name="front_bumper_link">
-    <pose>0 0 0 0 0 0</pose>
-    <collision name="front_bumper_col">
+  <link name="link_front_bumper">
+    <pose>0 0 0 0 0 0</pose>
+    <collision name="link_front_bumper_collision">
       <origin xyz="0 0 0" rpy="0 0 0"/>
       <geometry>

File: beacon_gazebo_plugin/urdf/autonet_v1/autonet_v1_gazebo.xacro (robot description, xacro)
@@ -6,10 +6,4 @@
   <gazebo reference="front_bumper_link">
     <material>Gazebo/White</material>
-  </gazebo>
-  <gazebo reference="link_left_wheel">
-    <material>Gazebo/Blue</material>
-  </gazebo>
-  <gazebo reference="link_right_wheel">
-    <material>Gazebo/Blue</material>
   </gazebo>
   <gazebo reference="receiver_link">
@@ -52,5 +46,13 @@
     </sensor>
   </gazebo>
-<!--  <gazebo reference="front_bumper_link">-->
+  <gazebo reference="link_front_bumper">
+<!--    <sensor name="my_contact" type="contact">-->
+<!--&lt;!&ndash;        <update_rate>1000</update_rate>&ndash;&gt;-->
+<!--&lt;!&ndash;        <always_on>true</always_on>&ndash;&gt;-->
+<!--        <contact>-->
+<!--          <collision>link_front_bumper_collision</collision>-->
+<!--        </contact>-->
+<!--    </sensor>-->
+  </gazebo>
 <!--&lt;!&ndash;    <sensor name='my_contact' type='contact'>&ndash;&gt;-->
 <!--&lt;!&ndash;      <update_rate>5</update_rate>&ndash;&gt;-->
@@ -94,5 +96,4 @@
 <!--&lt;!&ndash;      </controller:gazebo_ros_bumper>&ndash;&gt;-->
 <!--&lt;!&ndash;    </sensor:contact>&ndash;&gt;-->
-<!--  </gazebo>-->
   <gazebo reference="imu_link">
     <gravity>true</gravity>

File: beacon_gazebo_plugin/urdf/vc_robot_v1/macros.xacro (robot description, xacro)
@@ -25,5 +25,5 @@
                 </geometry>
             </collision>
-            <visual name="${name}_visual">
+            <visual name="link_${name}_wheel_visual">
                 <origin rpy="0 1.5707 1.5707" xyz="0 0 0"/>
                 <geometry>
@@ -32,15 +32,4 @@
             </visual>
         </link>
-        <gazebo reference="${name}">
-            <gravity>true</gravity>
-            <material>Gazebo/Grey</material>
-            <mu1>50</mu1>
-            <mu2>10</mu2>
-            <kp>10000000</kp>
-            <kd>1</kd>
-            <fdir1>1 0 0</fdir1>
-            <minDepth>0.0001</minDepth>
-            <maxContacts>1</maxContacts>
-        </gazebo>
     </xacro:macro>
     <xacro:macro name="joint_wheel" params="name child origin_xyz parent">
